Commit message: Completed Project Workspace

File: urdf/my_udacity_bot.xacro (robot description, xacro)
@@ -1,5 +1,5 @@
 <?xml version='1.0'?>
 <robot name="udacity_bot" xmlns:xacro="http://www.ros.org/wiki/xacro">
-<xacro:include filename="$(find udacity_bot)/urdf/udacity_bot.gazebo" />
+  <xacro:include filename="$(find udacity_bot)/urdf/my_udacity_bot.gazebo" />
   <link name="robot_footprint"></link>
   <joint name="robot_footprint_joint" type="fixed">
@@ -22,5 +22,5 @@
       <origin xyz="0 0 0" rpy=" 0 0 0"/>
       <geometry>
-        <box size=".4 .2 .1"/>
+        <box size=".2 .1 .05"/>
       </geometry>
     </collision>
@@ -28,12 +28,11 @@
       <origin xyz="0 0 0" rpy=" 0 0 0"/>
       <geometry>
-        <box size=".4 .2 .1"/>
+        <box size=".2 .1 .05"/>
       </geometry>
-    <material name="orange"/>
     </visual>
     <collision name='back_caster_collision'>
-      <origin xyz="-0.15 0 -0.05" rpy=" 0 0 0"/>
+      <origin xyz="-0.075 0 -0.025" rpy=" 0 0 0"/>
       <geometry>
-        <sphere radius="0.05"/>
+        <sphere radius="0.025"/>
       </geometry>
       <surface>
@@ -42,5 +41,5 @@
             <mu>0</mu>
             <mu2>0</mu2>
-            <slip1>1.0</slip1>
+            <slip1>.9</slip1>
             <slip2>1.0</slip2>
           </ode>
@@ -49,13 +48,13 @@
     </collision>
     <visual name='back_caster_visual'>
-      <origin xyz="-0.15 0 -0.05" rpy=" 0 0 0"/>
+      <origin xyz="-0.075 0 -0.025" rpy=" 0 0 0"/>
       <geometry>
-        <sphere radius="0.05"/>
+        <sphere radius="0.025"/>
       </geometry>
     </visual>
     <collision name='front_caster_collision'>
-      <origin xyz="0.15 0 -0.05" rpy=" 0 0 0"/>
+      <origin xyz="0.075 0 -0.025" rpy=" 0 0 0"/>
       <geometry>
-        <sphere radius="0.05"/>
+        <sphere radius="0.025"/>
       </geometry>
       <surface>
@@ -64,5 +63,5 @@
             <mu>0</mu>
             <mu2>0</mu2>
-            <slip1>1.0</slip1>
+            <slip1>.9</slip1>
             <slip2>1.0</slip2>
           </ode>
@@ -71,14 +70,14 @@
     </collision>
     <visual name='front_caster_visual'>
-      <origin xyz="0.15 0 -0.05" rpy=" 0 0 0"/>
+      <origin xyz=".075 0 -.025" rpy=" 0 0 0"/>
       <geometry>
-        <sphere radius="0.05"/>
+        <sphere radius=".025"/>
       </geometry>
     </visual>
   </link>
-  <link name='left_wheel'>
+  <link name="left_wheel">
     <inertial>
       <mass value="5.0"/>
-      <origin xyz="0.0 0.0 0.0" rpy=" 0 1.5707 1.5707"/>
+      <origin xyz="0 0 0" rpy="0 1.5707 1.5707"/>
       <inertia
           ixx="0.1" ixy="0" ixz="0"
@@ -88,18 +87,18 @@
     </inertial>
     <collision name='collision'>
-      <origin xyz="0.0 0.0 0.0" rpy=" 0 1.5707 1.5707"/>
+      <origin xyz="0 0 0" rpy="0 1.5707 1.5707"/>
       <geometry>
-        <cylinder radius="0.1" length="0.05"/>
+        <cylinder radius="0.05" length="0.025"/>
       </geometry>
     </collision>
-    <visual name='left_wheel_visual'>
-      <origin xyz="0.0 0 0.0" rpy=" 0 1.5707 1.5707"/>
+    <visual name='chassis_visual'>
+      <origin xyz="0 0 0" rpy="0 1.5707 1.5707"/>
       <geometry>
-        <cylinder radius="0.1" length="0.05"/>
+        <cylinder radius="0.05" length="0.025"/>
       </geometry>
     </visual>
   </link>
   <joint type="continuous" name="left_wheel_hinge">
-    <origin xyz="0 0.15 0" rpy="0 0 0"/>
+    <origin xyz="0 0.075 0" rpy="0 0 0"/>
     <child link="left_wheel"/>
     <parent link="chassis"/>
@@ -108,8 +107,8 @@
     <joint_properties damping="1.0" friction="1.0"/>
   </joint>
-    <link name='right_wheel'>
+  <link name="right_wheel">
     <inertial>
       <mass value="5.0"/>
-      <origin xyz="0.0 0 0.0" rpy=" 0 1.5707 1.5707"/>
+      <origin xyz="0 0 0" rpy="0 1.5707 1.5707"/>
       <inertia
           ixx="0.1" ixy="0" ixz="0"
@@ -119,18 +118,18 @@
     </inertial>
     <collision name='collision'>
-      <origin xyz="0.0 0 0.0" rpy=" 0 1.5707 1.5707"/>
+      <origin xyz="0 0 0" rpy="0 1.5707 1.5707"/>
       <geometry>
-        <cylinder radius="0.1" length="0.05"/>
+        <cylinder radius="0.05" length="0.025"/>
       </geometry>
     </collision>
-    <visual name='right_wheel_visual'>
-      <origin xyz="0.0 0 0.0" rpy=" 0 1.5707 1.5707"/>
+    <visual name='chassis_visual'>
+      <origin xyz="0 0 0" rpy="0 1.5707 1.5707"/>
       <geometry>
-        <cylinder radius="0.1" length="0.05"/>
+        <cylinder radius="0.05" length="0.025"/>
       </geometry>
     </visual>
   </link>
   <joint type="continuous" name="right_wheel_hinge">
-    <origin xyz="0 -0.15 0" rpy="0 0 0"/>
+    <origin xyz="0 -0.075 0" rpy="0 0 0"/>
     <child link="right_wheel"/>
     <parent link="chassis"/>
@@ -139,9 +138,9 @@
     <joint_properties damping="1.0" friction="1.0"/>
   </joint>
-  <!-- Camera Sensor -->
+  <!-- CAMERA -->
   <link name='camera'>
     <inertial>
-      <mass value=".1"/>
-      <origin xyz="0.0 0.0 0.0" rpy=" 0 0 0"/>
+      <mass value="0.1"/>
+      <origin xyz="0 0 0" rpy="0 0 0"/>
       <inertia
           ixx="1e-6" ixy="0" ixz="0"
@@ -151,26 +150,27 @@
     </inertial>
     <collision name='collision'>
-      <origin xyz="0.0 0.0 0.0" rpy=" 0 0 0"/>
+      <origin xyz="0 0 0" rpy="0 0 0"/>
       <geometry>
-        <box size=".05 .05 .05"/>
+        <box size="0.025 0.025 0.025"/>
       </geometry>
     </collision>
-    <visual name='camera_visual'>
-      <origin xyz="0.0 0 0.0" rpy=" 0 0 0"/>
+    <visual name='chassis_visual'>
+      <origin xyz="0 0 0" rpy="0 0 0"/>
       <geometry>
-        <box size=".05 .05 .05"/>
+        <box size="0.025 0.025 0.025"/>
       </geometry>
     </visual>
   </link>
+  <!--joint type="continuous" name="left_wheel_hinge"-->
   <joint type="fixed" name="camera_joint">
-    <origin xyz=".2 0 0" rpy="0 0 0"/>
+    <origin xyz="0.1 0 0" rpy="0 0 0"/>
     <child link="camera"/>
     <parent link="chassis"/>
   </joint>
-    <!-- Laser Rangefinder -->
+  <!-- hokuyo -->
   <link name='hokuyo'>
     <inertial>
-      <mass value=".1"/>
-      <origin xyz="0.0 0.0 0.0" rpy=" 0 0 0"/>
+      <mass value="0.1"/>
+      <origin xyz="0 0 0" rpy="0 0 0"/>
       <inertia
           ixx="1e-6" ixy="0" ixz="0"
@@ -180,18 +180,18 @@
     </inertial>
     <collision name='collision'>
-      <origin xyz="0.0 0.0 0.0" rpy=" 0 0 0"/>
+      <origin xyz="0 0 0" rpy="0 0 0"/>
       <geometry>
-        <box size=".1 .1 .1"/>
+        <box size="0.1 0.1 0.1"/>
       </geometry>
     </collision>
-    <visual name='camera_visual'>
-      <origin xyz="0.0 0 0.0" rpy=" 0 0 0"/>
+    <visual name='chassis_visual'>
+      <origin xyz="0 0 0" rpy="0 0 0"/>
       <geometry>
         <mesh filename="package://udacity_bot/meshes/hokuyo.dae"/>
       </geometry>
-      </visual>
+    </visual>
   </link>
   <joint type="fixed" name="hokuyo_joint">
-    <origin xyz=".15 0 .1" rpy="0 0 0"/>
+    <origin xyz="0.075 0 0.05" rpy="0 0 0"/>
     <child link="hokuyo"/>
     <parent link="chassis"/>
